File: SecuritySystem.kicad_sch (KiCad schematic)
At the start: 16 parts, among them J7 Fingerprint Scanner Terminal, J8 Servo Terminal, J9 RFID Module Terminal, Q1 FDN340P, U3 ESP32-DEVKIT-V1

Commit message: updated gerber files
re-add of resistor footprints -- for some reason it was removed
re-add of the new pull-down resistor R27 -- for some reason it was not
in the schematic but it exists in pcb
Parts:
- added R27: 2.2k, Resistor_THT:R_Axial_DIN0207_L6.3mm_D2.5mm_P7.62mm_Horizontal, symbol Device:R
- R25: value 47 -> 100
Connections:
- net GND: now also R27.2
- net servo_switch: now also R27.1
Changed lines of the file:
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@@
+	)
+	(symbol
+		(lib_id "Device:R")
+		(at 165.1 99.06 0)
+		(unit 1)
+		(exclude_from_sim no)
+		(in_bom yes)
+		(on_board yes)
+		(dnp no)
+		(fields_autoplaced yes)
+		(property "Reference" "R27"
+			(at 167.64 97.7899 0)
+			(effects
+				(font
+					(size 1.27 1.27)
+				)
+				(justify left)
+			)
+		)
+		(property "Value" "2.2k"
+			(at 167.64 100.3299 0)
+			(effects
+				(font
+					(size 1.27 1.27)
+				)
+				(justify left)
+			)
+		)
+		(property "Footprint" "Resistor_THT:R_Axial_DIN0207_L6.3mm_D2.5mm_P7.62mm_Horizontal"
+			(at 163.322 99.06 90)
+			(effects
+				(font
+					(size 1.27 1.27)
+				)
+				(hide yes)
+			)
+		)
+		(property "Datasheet" "~"
+			(at 165.1 99.06 0)
+			(effects
+				(font
+					(size 1.27 1.27)
+				)
+				(hide yes)
+			)
+		)
+		(property "Description" "Resistor"
+			(at 165.1 99.06 0)
+			(effects
+				(font
+					(size 1.27 1.27)
+				)
+				(hide yes)
+			)
+		)
+		(pin "2"
+		)
+		(pin "1"
+		)
+		(instances
+			(project ""
+				(path "/93d943f8-2f1f-47af-8720-a5ac9ef9a0be/3d33b991-ebd3-47c2-b368-2e09482c4f58"
+					(reference "R27")
+					(unit 1)
+				)
+			)
+		)
 	)
 	(symbol
@@
 	)
 	(symbol
+		(lib_id "power:GND")
+		(at 165.1 102.87 0)
+		(unit 1)
+		(exclude_from_sim no)
+		(in_bom yes)
+		(on_board yes)
+		(dnp no)
+		(fields_autoplaced yes)
+		(property "Reference" "#PWR019"
+			(at 165.1 109.22 0)
+			(effects
+				(font
+					(size 1.27 1.27)
+				)
+				(hide yes)
+			)
+		)
+		(property "Value" "GND"
+			(at 165.1 107.95 0)
+			(effects
+				(font
+					(size 1.27 1.27)
+				)
+			)
+		)
+		(property "Footprint" ""
+			(at 165.1 102.87 0)
+			(effects
+				(font
+					(size 1.27 1.27)
+				)
+				(hide yes)
+			)
+		)
+		(property "Datasheet" ""
+			(at 165.1 102.87 0)
+			(effects
+				(font
+					(size 1.27 1.27)
+				)
+				(hide yes)
+			)
+		)
+		(property "Description" "Power symbol creates a global label with name \"GND\" , ground"
+			(at 165.1 102.87 0)
+			(effects
+				(font
+					(size 1.27 1.27)
+				)
+				(hide yes)
+			)
+		)
+		(pin "1"
+		)
+		(instances
+			(project ""
+				(path "/93d943f8-2f1f-47af-8720-a5ac9ef9a0be/3d33b991-ebd3-47c2-b368-2e09482c4f58"
+					(reference "#PWR019")
+					(unit 1)
+				)
+			)
+		)
+	)
+	(symbol
 		(lib_id "Device:R")
 		(at 114.3 90.17 90)
@@
 			)
 		)
-		(property "Value" "47"
+		(property "Value" "100"
 			(at 88.9 137.16 0)
 			(effects

Commit message: revision 2
modified pull-up/pull-down resistor values
modified switch1/switch2 input voltage from 5V to 3v3

added proper sheet detail (designer, cc license)
Parts:
- R27: value 2.2k -> 10k
Changed lines of the file:
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@@
 		(title "Multi-Layer Security System")
 		(date "2025-11-02")
-		(rev "0")
+		(rev "2")
+		(comment 1 "Designed by: Sidney Manzano")
+		(comment 2 "Released under the Creative Commons")
+		(comment 3 "Attribution Share-Alike 4.0 License")
+		(comment 4 "https://creativecommons.org/licenses/by-sa/4.0")
 	)
 	(junction
@@
 			)
 		)
-		(property "Value" "2.2k"
+		(property "Value" "10k"
 			(at 167.64 100.3299 0)
 			(effects
